File: ALTAIR_SERVO_MODULE_V5/ALTAIR_SERVO_MODULE_V5.kicad_sch (KiCad schematic)
At the start: 53 parts, among them IC1 TLP152, IC2 TLP152, IC3 TLP152, IC4 TLP152, IC5 TLP152, IC6 TLP152, IC7 TLP152, IC8 TLP152, J1 servo, J11 USB_A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

Commit message: Add files via upload
Parts:
- IC1, IC2, IC3, IC4, IC5, IC6, IC7, IC8: value TLP152 -> TLP2304
Other:
- title: ALTAIR_SERVO_MODULE_V2 -> ALTAIR_SERVO_MODULE_V5
Changed lines of the file:
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@@
 	(paper "User" 297.002 212.319)
 	(title_block
-		(title "ALTAIR_SERVO_MODULE_V2")
-		(date "2024-02-26")
+		(title "ALTAIR_SERVO_MODULE_V5")
+		(date "2025-03-01")
 		(rev "2.0.0")
 		(company "-Altair-")
@@
 		(fields_autoplaced yes)
 		(property "Reference" "IC2"
-			(at 70.485 76.835 0)
+			(at 70.485 77.47 0)
 			(effects
 				(font
@@
 			)
 		)
-		(property "Value" "TLP152"
-			(at 70.485 79.375 0)
+		(property "Value" "TLP2304"
+			(at 70.485 80.01 0)
 			(effects
 				(font
@@
 		(fields_autoplaced yes)
 		(property "Reference" "IC3"
-			(at 70.485 93.345 0)
+			(at 70.485 93.98 0)
 			(effects
 				(font
@@
 			)
 		)
-		(property "Value" "TLP152"
-			(at 70.485 95.885 0)
+		(property "Value" "TLP2304"
+			(at 70.485 96.52 0)
 			(effects
 				(font
@@
 			)
 		)
-		(property "Value" "TLP152"
+		(property "Value" "TLP2304"
 			(at 70.485 113.03 0)
 			(effects
@@
 			)
 		)
-		(property "Value" "TLP152"
+		(property "Value" "TLP2304"
 			(at 70.485 163.83 0)
 			(effects
@@
 		(fields_autoplaced yes)
 		(property "Reference" "IC6"
-			(at 70.485 144.145 0)
+			(at 70.485 144.78 0)
 			(effects
 				(font
@@
 			)
 		)
-		(property "Value" "TLP152"
-			(at 70.485 146.685 0)
+		(property "Value" "TLP2304"
+			(at 70.485 147.32 0)
 			(effects
 				(font
@@
 			)
 		)
-		(property "Value" "TLP152"
+		(property "Value" "TLP2304"
 			(at 69.85 62.23 0)
 			(effects
@@
 		(fields_autoplaced yes)
 		(property "Reference" "IC8"
-			(at 70.485 178.435 0)
+			(at 70.485 179.07 0)
 			(effects
 				(font
@@
 			)
 		)
-		(property "Value" "TLP152"
-			(at 70.485 180.975 0)
+		(property "Value" "TLP2304"
+			(at 70.485 181.61 0)
 			(effects
 				(font
@@
 			)
 		)
-		(property "Value" "TLP152"
+		(property "Value" "TLP2304"
 			(at 70.485 129.54 0)
 			(effects
